File: pcb2/avm1c_pcb2.kicad_pcb (KiCad board)
At the start: 2 copper layers, 37.5 x 100 mm, 39 parts, among them J12 Conn_01x08, J13 Conn_01x06, J14 Conn_01x08, J16 Conn_01x04, J3 Conn_Coaxial, J4 Conn_Coaxial, J9 Eurorack_Header_LZX, M3 MountingHole_3.2mm_M3_9mm_cle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, U1 LM6172, U2 MCP6002-xP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

Commit message: Updated board after upgrading kicad
Parts:
- C3, C4: value 100nf -> 100nF
- moved C3 2.65 mm to (39.8, 55.3), turned to 90 degrees
- moved C4 2.53 mm to (32.2, 50.7), turned to 90 degrees
Connections:
- C4 pad 1: GND -> Net-(C4-Pad1)
- C4 pad 2: Net-(C4-Pad2) -> GND
- J3 pad 1: Net-(C3-Pad2) -> Net-(C3-Pad1)
- J4 pad 1: Net-(C3-Pad2) -> Net-(C3-Pad1)
- JP2 pad 2: Net-(C3-Pad2) -> Net-(C3-Pad1)
- R11 pad 2: Net-(C4-Pad2) -> Net-(C4-Pad1)
- U3 pad 2: Net-(C3-Pad1) -> Net-(C3-Pad2)
- U3 pad 6: Net-(C4-Pad2) -> Net-(C4-Pad1)
Routing:
- net Net-(C3-Pad2): track 27.0 -> 4.11 mm
- net Net-(C3-Pad1): track 4.11 -> 27.0 mm
- net Net-(C4-Pad2): track 5.71 -> 0.00 mm
- net Net-(C4-Pad1): track 0.00 -> 5.71 mm
Other:
- board text added: "TODO: Replace the DIP LM1881 with a SOIC one! (or a dual format footprint?)"
