File: combined_schematic/avm1c_combined_schematic.sch (KiCad schematic (older format))
At the start: 66 parts, among them J1 Video_Output, J2 Jack_X_CV, J3 Conn_Coaxial, J4 Conn_Coaxial, J5 Jack_Y_CV, J6 Jack_Index_CV, J8 Jack_Trigger, J9 Eurorack_Header_LZX, Q1 2N3904, SW1 Button_Mode, SW2 Button_Trigger, SW3 Button_Arduino_Reset, U1 LM6172, U2 MCP6002-xP, U3 LM1881, U5 MCP6002-xP, U6 L7805, U7 LM4040LP-5

Commit message: Updated board after upgrading kicad
Changed lines of the file:
@@
 EESchema Schematic File Version 4
-LIBS:avm1c_combined_schematic-cache
-EELAYER 29 0
+EELAYER 30 0
 EELAYER END
 $Descr USLedger 11000 17000 portrait
@@
 NoConn ~ 950  9650
 $Comp
-L MCU_Module:Arduino_Nano_v3.x A?
-U 1 1 6058E8FF
-P 3300 9050
-AR Path="/5E6B5FB1/6058E8FF" Ref="A?"  Part="1"
-AR Path="/6058E8FF" Ref="A1"  Part="1"
-F 0 "A1" H 2800 8050 50  0000 C CNN
-F 1 "Arduino_Nano_v3.x" H 2750 7950 50  0000 C CNN
-F 2 "Module:Arduino_Nano" H 3450 8100 50  0001 L CNN
-F 3 "http://www.mouser.com/pdfdocs/Gravitech_Arduino_Nano3_0.pdf" H 3300 8050 50  0001 C CNN
-	1    3300 9050
-	1    0    0    -1
-$EndComp
-$Comp
 L power:+5V #PWR?
 U 1 1 6058E905
@@
 Text Notes 8150 13650 0    100  ~ 0
 Unused Op Amp in LM6172
+$Comp
+L MCU_Module:Arduino_Nano_v3.x A1
+U 1 1 6173A9AE
+P 3300 9050
+F 0 "A1" H 3050 7950 50  0000 C CNN
+F 1 "Arduino_Nano_v3.x" H 2900 7850 50  0000 C CNN
+F 2 "Module:Arduino_Nano" H 3300 9050 50  0001 C CIN
+F 3 "http://www.mouser.com/pdfdocs/Gravitech_Arduino_Nano3_0.pdf" H 3300 9050 50  0001 C CNN
+	1    3300 9050
+	1    0    0    -1
+$EndComp
 $EndSCHEMATC

Commit message: fix combined schematic and pcb
Parts:
- added H1, H2: MountingHole, MountingHole:MountingHole_3.2mm_M3, symbol Mechanical:MountingHole
- added J10: Front_Conn_1, Connector_PinHeader_2.54mm:PinHeader_1x08_P2.54mm_Vertical, symbol Connector_Generic:Conn_01x08
- added J11: Front_Conn_3, Connector_PinHeader_2.54mm:PinHeader_1x06_P2.54mm_Vertical, symbol Connector_Generic:Conn_01x06
- added J12: Back_Conn_2, Connector_PinSocket_2.54mm:PinSocket_1x08_P2.54mm_Vertical, symbol Connector_Generic:Conn_01x08
- added J13: Back_Conn_3, Connector_PinSocket_2.54mm:PinSocket_1x06_P2.54mm_Vertical, symbol Connector_Generic:Conn_01x06
- added J14: Back_Conn_1, Connector_PinSocket_2.54mm:PinSocket_1x08_P2.54mm_Vertical, symbol Connector_Generic:Conn_01x08
- added J15: Front_Conn_4, Connector_PinHeader_2.54mm:PinHeader_1x04_P2.54mm_Vertical, symbol Connector_Generic:Conn_01x04
- added J16: Back_Conn_4, Connector_PinSocket_2.54mm:PinSocket_1x04_P2.54mm_Vertical, symbol Connector_Generic:Conn_01x04
- added J17: VIN, Connector_Wire:SolderWire-0.5sqmm_1x01_D0.9mm_OD2.1mm, symbol Connector_Generic:Conn_01x01
- added J7: Front_Conn_2, Connector_PinHeader_2.54mm:PinHeader_1x08_P2.54mm_Vertical, symbol Connector_Generic:Conn_01x08
Connections:
- net +5V: now also J13.1 (Pin_1), J13.2 (Pin_2); no longer C9.1, R25.2, RV1.1, RV2.1, RV3.1, U5.6 (-), U5.8 (V+)
- net -12V: now also J14.4 (Pin_4); no longer R28.1
- net VIDEO_OUT_POST_BACK: now reaches R5.2, U1.1
- net VIDEO_OUT_POST_BACK: now also J14.3 (Pin_3); no longer R2.2
- net X_CV_PRE_BACK: now reaches C1.2, R7.2, U2.2 (-)
- net X_CV_PRE_BACK: now also J13.4 (Pin_4); no longer R3.1, R6.1, R8.1
- net Y_CV_PRE_BACK: now reaches C2.2, R15.2, U2.6 (-)
- net Y_CV_PRE_BACK: now also J13.3 (Pin_3); no longer R13.1, R14.1, R16.1
- net at A1.30 (VIN): now also J17.1 (Pin_1)
- net GND renamed GND2
- net GND2: now also J12.1 (Pin_1), J12.2 (Pin_2), J12.5 (Pin_5), J12.6 (Pin_6), J12.7 (Pin_7), J12.8 (Pin_8), J13.5 (Pin_5), J13.6 (Pin_6), J14.1 (Pin_1), J14.2 (Pin_2), J14.7 (Pin_7), J14.8 (Pin_8), J16.2 (Pin_2), J16.3 (Pin_3), J16.4 (Pin_4); no longer C13.2, C9.2, D3.2 (A), J1.S, J2.S, J5.S, J6.S, J8.S, Q1.1 (E), RV1.3, RV2.3, RV3.3, SW1.1, SW2.1, SW3.1, U5.3 (+), U5.4 (V-), U5.5 (+), U7.2 (K)
- net INDEX_CV renamed INDEX_CV_FRONT
- net INDEX_CV_FRONT: now also J7.4 (Pin_4); no longer A1.19 (A0)
- net MODE_SWITCH renamed MODE_SWITCH_BACK
- net MODE_SWITCH_BACK: now also J14.5 (Pin_5); no longer SW1.2
- net RESET_SWITCH renamed RESET_SWITCH_BACK
- net RESET_SWITCH_BACK: now also J16.1 (Pin_1); no longer SW3.2
- net TRIGGER_CV renamed TRIGGER_CV_FRONT
- net TRIGGER_CV_FRONT: now also J10.6 (Pin_6); no longer A1.13 (D10)
- net TRIGGER_SWITCH renamed TRIGGER_SWITCH_BACK
- net TRIGGER_SWITCH_BACK: now also J12.3 (Pin_3); no longer SW2.2
- new net +5VA: C9.1, J11.1 (Pin_1), J11.2 (Pin_2), R25.2, RV1.1, RV2.1, RV3.1, U5.6 (-), U5.8 (V+)
- new net GND1: C13.2, C9.2, D3.2 (A), J1.S, J10.1 (Pin_1), J10.2 (Pin_2), J10.7 (Pin_7), J10.8 (Pin_8), J11.5 (Pin_5), J11.6 (Pin_6), J15.2 (Pin_2), J15.3 (Pin_3), J15.4 (Pin_4), J2.S, J5.S, J6.S, J7.1 (Pin_1), J7.2 (Pin_2), J7.5 (Pin_5), J7.6 (Pin_6), J7.7 (Pin_7), J7.8 (Pin_8), J8.S, Q1.1 (E), RV1.3, RV2.3, RV3.3, SW1.1, SW2.1, SW3.1, U5.3 (+), U5.4 (V-), U5.5 (+), U7.2 (K)
- new net INDEX_CV_BACK: A1.19 (A0), J12.4 (Pin_4)
- new net MODE_SWITCH_FRONT: J10.5 (Pin_5), SW1.2
- new net RESET_SWITCH_FRONT: J15.1 (Pin_1), SW3.2
- new net TRIGGER_CV_BACK: A1.13 (D10), J14.6 (Pin_6)
- new net TRIGGER_SWITCH_FRONT: J7.3 (Pin_3), SW2.2
- new net VEE: J10.4 (Pin_4), R28.1
- new net VIDEO_OUT_POST_FRONT: J10.3 (Pin_3), R2.2
- new net X_CV_PRE_FRONT: J11.4 (Pin_4), R3.1, R6.1, R8.1
- new net Y_CV_PRE_FRONT: J11.3 (Pin_3), R13.1, R14.1, R16.1
- no-connect marks 26 -> 25
Other:
- note added: "(-12V)"
- note added: "+5VA is the +5V on PCB1\nVEE is the -12V on PCB1\nGND1 is the GND on PCB1\n\nGND2 is the GND on PCB2\n+5V is the +5V on PCB2\n-12V is the -12V on PCB2\n+12V is the +12V on PCB2\n"
- note added: "MCP6002 Power and Bypass Cap"
- moved on the sheet: A1, C1, C10, C11, C12, C13, C14, C15, C2, C3, C4, C5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
