File: pcb/avm1c_combined_schematic.kicad_pcb (KiCad board)
At the start: 2 copper layers, 100.6 x 100 mm, 81 parts, among them J1 Video_Output, J10 Front_Conn_1, J11 Front_Conn_3, J12 Back_Conn_2, J13 Back_Conn_3, J14 Back_Conn_1, J15 Front_Conn_4, J16 Back_Conn_4, J17 VIN, J2 Jack_X_CV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

Commit message: Add todo note to drawings layer
Other:
- board text added: "TODO: Add 3D models for the jacks and arduino!"
