File: panel/avml_panel.kicad_pcb (KiCad board)
At the start: 2 copper layers, 40.3 x 128.5 mm, 13 parts, among them J1 DNP

Commit message: Update panel to kicad 6+
Other:
- net class Default removed
